File: Left.kicad_sch (KiCad schematic)
At the start: 206 parts

Commit message: "Finalized" the schematics
Reorganized schematics, finished up the matrixes with correct number of switches and LEDs, other minor tasks
Parts:
- removed D? (x6): (no value), symbol Device:LED
- removed D? (x7): (no value), symbol Device:D_Small
- removed R? (x6): (no value), symbol Device:R_Small
- removed SW? (x7): (no value), symbol Switch:SW_Push
- added D4, D61: LED, symbol Device:LED
- added D47, D48: D_Small, symbol Device:D_Small
- added Q2: DMN2041L, Package_TO_SOT_SMD:SOT-23, symbol Transistor_FET:DMN2041L
- added R5, R50: 470, symbol Device:R_Small
- added R51: 1k, symbol Device:R_Small
- added R52, R53: 5.1k, symbol Device:R_Small
- added SW7, SW8: SW_Push, keyswitches.pretty-2:Kailh_socket_PG1350, symbol Switch:SW_Push
- C1, C2: renamed from C?; value (none) -> 22pF
- C3: renamed from C?; value (none) -> 1uF
- C4, C5, C6: renamed from C?; value (none) -> .1uF
- C7: renamed from C?; value (none) -> 10uf
- D1: renamed from D?; value (none) -> PRTR5V0U2X; footprint (none) -> Package_TO_SOT_SMD:SOT-143
- D10, D11, D12, D13, D14, D15, D16, D17, D18, D19, D2, D20, D21, D22, D23, D24, D25, D26, D27, D28, D29, D3, D30, D31, D32, D33, D34, D35, D36, D37, D38, D39, D40, D41, D5, D6, D7, D8, D9: renamed from D?; value (none) -> LED
- D42, D43, D44, D45, D46, D49, D50, D51, D52, D53, D54, D55, D56, D57, D58, D59, D60, D62, D63, D64, D65, D66, D67, D68, D69, D70, D71, D72, D73, D74, D75, D76, D77, D78, D79, D80, D81, D82: renamed from D?; value (none) -> D_Small
- F1: renamed from F?; value (none) -> 500m
- J1, J2: renamed from J?; value (none) -> USB_C_Receptacle_USB2.0
- J3: renamed from J?; value (none) -> AVR-ISP-6
- Q1: renamed from Q?; value (none) -> DMN2041L; footprint (none) -> Package_TO_SOT_SMD:SOT-23
- R1, R2: renamed from R?; value (none) -> 5.1k
- R10, R11, R12, R13, R14, R15, R16, R17, R19, R20, R21, R24, R25, R26, R27, R28, R29, R3, R30, R31, R32, R33, R34, R35, R37, R38, R39, R4, R42, R43, R44, R45, R46, R47, R48, R6, R7, R8, R9: renamed from R?; value (none) -> 470
- R18, R22: renamed from R?; value (none) -> 22
- R23, R36: renamed from R?; value (none) -> 10k
- R40, R41: renamed from R?; value (none) -> 4.7K
- R49: renamed from R?; value (none) -> 1k
- SW1: renamed from SW?; value (none) -> RotaryEncoder
- SW10, SW11, SW12, SW13, SW14, SW15, SW16, SW17, SW18, SW19, SW2, SW20, SW21, SW22, SW23, SW24, SW25, SW26, SW27, SW28, SW29, SW3, SW30, SW31, SW32, SW33, SW34, SW35, SW36, SW37, SW38, SW39, SW4, SW40, SW41, SW5, SW6, SW9: renamed from SW?; value (none) -> SW_Push; footprint (none) -> keyswitches.pretty-2:Kailh_socket_PG1350
- SW_RESET1: renamed from SW?; value (none) -> SW_Push; footprint (none) -> Button_Switch_SMD:SW_SPST_SKQG_WithStem
- U1: renamed from U?; value (none) -> ATmega32U4-A; footprint (none) -> ATmega32U4:ATmega32U4
- Y1: renamed from Y?; value (none) -> 16MHz
Connections:
- net +5V: now also D4.2 (A), D61.2 (A)
- net COL_1: now also SW7.2, SW8.2
- net GND: now also Q2.2 (S), R52.2, R53.2
- net ROW_5: now also D48.1 (K)
- net ROW_6: now also D47.1 (K)
- net at Q1.3 (D), R10.2, R11.2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: now also R5.2
- net at J1.A5 (CC1): now also R53.1
- net at J1.B5 (CC2): now also R52.1
- net CAPS_LOCK_PWM: now reaches U1.31 (PC6)
- net CAPS_LOCK_PWM: now also R51.2
- new net: D61.1 (K), R50.1
- new net: Q2.1 (G), R51.1
- new net: Q2.3 (D), R50.2
- new net: D48.2 (A), SW8.1
- new net: D47.2 (A), SW7.1
- new net: D4.1 (K), R5.1
- no-connect marks 3 -> 8
Other:
- note added: "40 LEDs"
- note added: "40 switch matrix"
- note added: "CAPS LOCK LED"
- note added: "LEFT KEEEB HALF"
- note added: "MCU"
- note added: "USB-C RIGHT HALF"
- note removed: "39"
- note removed: "LEDs"
- moved on the sheet: C1, C2, C3, C4, C5, C6, C7, D1, D10, D11, D12, D13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
