File: Right.kicad_sch (KiCad schematic)
At the start: 206 parts, among them J1 USB_C_Receptacle_USB2.0, J2 USB_C_Receptacle_USB2.0, J3 AVR-ISP-6, Q1 DMN2041L, SW1 SW_Push, SW10 SW_Push, SW11 SW_Push, SW12 SW_Push, SW13 SW_Push, SW14 SW_Push, SW15 SW_Push, SW16 SW_Push, SW17 SW_Push, SW18 SW_Push, SW19 SW_Push, SW2 SW_Push, SW20 SW_Push, SW21 SW_Push, SW22 SW_Push, SW23 SW_Push, SW24 SW_Push, SW25 SW_Push, SW26 SW_Push, SW27 SW_Push, SW28 SW_Push, SW29 RotaryEncoder, SW3 SW_Push, SW30 SW_Push, SW31 SW_Push, SW32 SW_Push, SW33 SW_Push, SW34 SW_Push, SW35 SW_Push, SW36 SW_Push, SW37 SW_Push, SW38 SW_Push, SW39 SW_Push, SW4 SW_Push, SW40 SW_Push, SW41 SW_Push, SW42 SW_Push, SW43 SW_Push, SW44 SW_Push, SW45 SW_Push, SW46 SW_Push, SW47 SW_Push, SW5 SW_Push, SW6 SW_Push, SW7 SW_Push, SW8 SW_Push, SW9 SW_Push, U1 ATmega32U4-A, Y1 16MHz

Commit message: "Finalized" the schematics
Reorganized schematics, finished up the matrixes with correct number of switches and LEDs, other minor tasks
Parts:
- removed D22, D32, D36, D65: LED, symbol Device:LED
- removed D26, D38, D53, D55, D59: D_Small, symbol Device:D_Small
- removed SW16, SW19, SW22, SW26: SW_Push, symbol Switch:SW_Push
- removed SW29: RotaryEncoder, symbol Device:RotaryEncoder
- added D22: D_Small, symbol Device:D_Small
- added D26: LED, symbol Device:LED
- added Q2: DMN2041L, Package_TO_SOT_SMD:SOT-23, symbol Transistor_FET:DMN2041L
- C1, C2, C7: value .1uF -> (none)
- C3, C5: value 22pF -> (none)
- C4: value 1uF -> (none)
- C6: value 10uf -> (none)
- D1, D11, D14, D17, D18, D19, D2, D20, D3, D31, D33, D34, D35, D39, D40, D44, D46, D48, D50, D52, D56, D61, D62, D63, D64, D67, D7, D72, D73, D74, D75, D76, D79, D8, D82, D83, D85, D86, D88, D9, D91: value LED -> (none)
- D12, D13, D15, D16, D23, D24, D25, D27, D28, D29, D30, D37, D41, D42, D43, D45, D47, D49, D5, D51, D54, D57, D58, D6, D60, D66, D68, D69, D70, D71, D77, D78, D80, D81, D84, D87, D89, D90: value D_Small -> (none)
- D21: value PRTR5V0U2X -> (none); footprint Package_TO_SOT_SMD:SOT-143 -> (none)
- F1: value 500m -> (none)
- J1, J2: value USB_C_Receptacle_USB2.0 -> (none)
- J3: value AVR-ISP-6 -> (none)
- Q1: value DMN2041L -> (none); footprint Package_TO_SOT_SMD:SOT-23 -> (none)
- R1, R11, R12, R13, R14, R15, R17, R18, R19, R20, R24, R25, R27, R28, R29, R3, R30, R33, R35, R36, R37, R38, R39, R4, R40, R41, R42, R43, R45, R46, R47, R48, R49, R5, R50, R52, R53, R54, R6, R7, R9: value 470 -> (none)
- R10: value 470 -> 1k
- R16, R26: value 4.7K -> (none)
- R2, R44: value 22 -> (none)
- R21: value 1k -> (none)
- R22, R31: value 5.1k -> (none)
- R23, R34: value 10k -> (none)
- R32, R51: value 470 -> 5.1k
- SW1, SW10, SW11, SW12, SW13, SW14, SW15, SW17, SW18, SW2, SW20, SW21, SW23, SW24, SW25, SW27, SW30, SW31, SW32, SW33, SW34, SW35, SW36, SW37, SW38, SW39, SW4, SW40, SW41, SW42, SW43, SW44, SW45, SW46, SW47, SW5, SW6, SW7: value SW_Push -> (none); footprint (none) -> keyswitches.pretty-2:Kailh_socket_PG1350
- SW3, SW8, SW9: footprint (none) -> keyswitches.pretty-2:Kailh_socket_PG1350
- SW_RESET1: renamed from SW28; value SW_Push -> (none); footprint Button_Switch_SMD:SW_SPST_SKQG_WithStem -> (none)
- U1: value ATmega32U4-A -> (none); footprint ATmega32U4:ATmega32U4 -> (none)
- Y1: value 16MHz -> (none)
Connections:
- net +5V: now also D26.2 (A)
- net COL_0: now also SW3.2
- net COL_1: now also SW8.2, SW9.2
- net GND: now also R32.2, R51.2, Q2.2 (S)
- net ROW_2: no longer D10.1 (K)
- net ROW_5: now also D4.1 (K), D22.1 (K)
- net ROW_6: now also D10.1 (K); no longer D4.1 (K)
- net CAPS_LOCK_PWM: now reaches U1.31 (PC6)
- net CAPS_LOCK_PWM: now also R10.2
- net at Q1.3 (D), R1.2, R11.2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: no longer R10.2, R32.2, R51.2, R8.2
- net at D4.2 (A): now also SW3.1
- net at D10.2 (A): now also SW8.1; no longer SW9.1
- net at R8.1: now also D26.1 (K)
- net at R10.1: now also Q2.1 (G)
- net at R51.1: now also J2.A5 (CC1)
- net at J2.B5 (CC2): now also R32.1
- removed net COL_6: SW3.2, SW8.2, SW9.2
- net ENC_A: no longer names the net of U1.18 (PD0)
- net ENC_B: no longer names the net of U1.19 (PD1)
- new net: Q2.3 (D), R8.2
- new net: D22.2 (A), SW9.1
- no-connect marks 3 -> 10
Other:
- note added: "41 LEDs"
- note added: "41 switch matrix"
- note added: "CAPS LOCK LED"
- note added: "MCU"
- note added: "RIGHT KEEB HALF"
- note added: "USB-C Left HALF"
- note removed: "39"
- note removed: "LEDs"
- note removed: "Scroll Drum"
- moved on the sheet: C1, C2, C3, C4, C5, C6, C7, D1, D11, D12, D13, D14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

Commit message: Added ESD to half connectors, other changes too
Parts:
- added D?: PRTR5V0U2X, Package_TO_SOT_SMD:SOT-143, symbol Power_Protection:PRTR5V0U2X
- C1, C2, C7: value (none) -> .1uF
- C3, C5: value (none) -> 22pF
- C4: value (none) -> 1uF
- C6: value (none) -> 10uf
- D1, D11, D14, D17, D18, D19, D2, D20, D3, D31, D33, D34, D35, D39, D40, D44, D46, D48, D50, D52, D56, D61, D62, D63, D64, D67, D7, D72, D73, D74, D75, D76, D79, D8, D82, D83, D85, D86, D88, D9, D91: value (none) -> LED
- D12, D13, D15, D16, D23, D24, D25, D27, D28, D29, D30, D37, D41, D42, D43, D45, D47, D49, D5, D51, D54, D57, D58, D6, D60, D66, D68, D69, D70, D71, D77, D78, D80, D81, D84, D87, D89, D90: value (none) -> D_Small
- D21: value (none) -> PRTR5V0U2X; footprint (none) -> Package_TO_SOT_SMD:SOT-143
- F1: value (none) -> 500m
- J1, J2: value (none) -> USB_C_Receptacle_USB2.0
- J3: value (none) -> AVR-ISP-6
- Q1: value (none) -> DMN2041L; footprint (none) -> Package_TO_SOT_SMD:SOT-23
- R1, R11, R12, R13, R14, R15, R17, R18, R19, R20, R24, R25, R27, R28, R29, R3, R30, R33, R35, R36, R37, R38, R39, R4, R40, R41, R42, R43, R45, R46, R47, R48, R49, R5, R50, R52, R53, R54, R6, R7, R9: value (none) -> 470
- R16, R26: value (none) -> 4.7K
- R2, R44: value (none) -> 22
- R21: value (none) -> 1k
- R22, R31: value (none) -> 5.1k
- R23, R34: value (none) -> 10k
- SW1, SW10, SW11, SW12, SW13, SW14, SW15, SW17, SW18, SW2, SW20, SW21, SW23, SW24, SW25, SW27, SW30, SW31, SW32, SW33, SW34, SW35, SW36, SW37, SW38, SW39, SW4, SW40, SW41, SW42, SW43, SW44, SW45, SW46, SW47, SW5, SW6, SW7: value (none) -> SW_Push
- SW_RESET1: value (none) -> SW_Push; footprint (none) -> Button_Switch_SMD:SW_SPST_SKQG_WithStem
- U1: value (none) -> ATmega32U4-A; footprint (none) -> ATmega32U4:ATmega32U4
- Y1: value (none) -> 16MHz
Connections:
- net +5V: now also D?.4 (VCC)
- net DATA_1: now also D?.3 (I/O2)
- net GND: now also D?.1 (GND)
Other:
- note added: "RIGHT KEEEB HALF"
- note removed: "RIGHT KEEB HALF"
- moved on the sheet: C1, C2, C6, C7, D21, F1, J1, J2, J3, R22, R31, R32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
