File: halfjunk.kicad_pcb (KiCad board)
At the start: 2 copper layers, 369.1 x 95.2 mm, 92 parts

Commit message: replaced LEDs with RGBs, and started the PCB for keyboard
Parts:
- removed ATmega32U4: VAL**, ATmega32U4:ATmega32U4
- removed LED4: WS2812B, Keebio-Parts:WS2812B
- removed REF** (x81): SW_PG1350, keyswitches.pretty-2:SW_PG1350
- removed REF** (x4): USB_C_Receptacle_HRO_TYPE-C-31-M-12, Connector_USB:USB_C_Receptacle_HRO_TYPE-C-31-M-12
- removed REF**: RollerEncoder_Panasonic_EVQWGD001, rollyboi9000000-main:RollerEncoder_Panasonic_EVQWGD001
- removed REF** (x2): SW_SPST_SKQG_WithStem, Button_Switch_SMD:SW_SPST_SKQG_WithStem
- removed REF**: SK6812-MINI-E, Keebio-Parts:SK6812-MINI-E
- removed REF**: RotaryEncoder_Alps_EC11E-Switch_Vertical_H20mm, Rotary_Encoder:RotaryEncoder_Alps_EC11E-Switch_Vertical_H20mm
- added C201: 22pF, Capacitor_SMD:C_0402_1005Metric, B.Cu at (-100.5, 113.0)
- added C202: 22pF, Capacitor_SMD:C_0402_1005Metric, B.Cu at (-101.5, 109.0)
- added C203: 1uF, Capacitor_SMD:C_0402_1005Metric, B.Cu at (-120.5, 93.0)
- added C204: .1uF, Capacitor_SMD:C_0402_1005Metric, B.Cu at (-104.5, 96.0)
- added C205: .1uF, Capacitor_SMD:C_0402_1005Metric, B.Cu at (-124.5, 126.0)
- added C206: .1uF, Capacitor_SMD:C_0402_1005Metric, B.Cu at (-108.5, 96.0)
- added C207: 10uf, Capacitor_SMD:C_0402_1005Metric, B.Cu at (-109.5, 93.0)
- added C208: 100nF, Capacitor_SMD:C_0402_1005Metric, B.Cu at (309.9, 231.0)
- added C209: 100nF, Capacitor_SMD:C_0402_1005Metric, B.Cu at (289.8, 225.1)
- added C210: 100nF, Capacitor_SMD:C_0402_1005Metric, B.Cu at (307.0, 225.1)
- added C211: 100nF, Capacitor_SMD:C_0402_1005Metric, B.Cu at (301.3, 233.0)
- added C212: 100nF, Capacitor_SMD:C_0402_1005Metric, B.Cu at (307.0, 229.0)
- added C213: 100nF, Capacitor_SMD:C_0402_1005Metric, B.Cu at (298.4, 227.1)
- added C214: 100nF, Capacitor_SMD:C_0402_1005Metric, B.Cu at (289.8, 223.1)
- added C215: 100nF, Capacitor_SMD:C_0402_1005Metric, B.Cu at (307.0, 231.0)
- added C216: 100nF, Capacitor_SMD:C_0402_1005Metric, B.Cu at (298.4, 231.0)
- added C217: 100nF, Capacitor_SMD:C_0402_1005Metric, B.Cu at (304.1, 231.0)
- added C218: 100nF, Capacitor_SMD:C_0402_1005Metric, B.Cu at (295.5, 227.1)
- added C219: 100nF, Capacitor_SMD:C_0402_1005Metric, B.Cu at (295.5, 225.1)
- added C220: 100nF, Capacitor_SMD:C_0402_1005Metric, B.Cu at (304.1, 227.1)
- added C221: 100nF, Capacitor_SMD:C_0402_1005Metric, B.Cu at (309.9, 227.1)
- added C222: 100nF, Capacitor_SMD:C_0402_1005Metric, B.Cu at (301.3, 223.1)
- added C223: 100nF, Capacitor_SMD:C_0402_1005Metric, B.Cu at (301.3, 225.1)
- added C224: 100nF, Capacitor_SMD:C_0402_1005Metric, B.Cu at (307.0, 233.0)
- added C225: 100nF, Capacitor_SMD:C_0402_1005Metric, B.Cu at (309.9, 223.1)
- added C226: 100nF, Capacitor_SMD:C_0402_1005Metric, B.Cu at (295.5, 231.0)
- added C227: 100nF, Capacitor_SMD:C_0402_1005Metric, B.Cu at (307.0, 227.1)
- added C228: 100nF, Capacitor_SMD:C_0402_1005Metric, B.Cu at (309.9, 225.1)
- added C229: 100nF, Capacitor_SMD:C_0402_1005Metric, B.Cu at (292.6, 227.1)
- added C230: 100nF, Capacitor_SMD:C_0402_1005Metric, B.Cu at (304.1, 225.1)
- added C231: 100nF, Capacitor_SMD:C_0402_1005Metric, B.Cu at (301.3, 229.0)
- added C232: 100nF, Capacitor_SMD:C_0402_1005Metric, B.Cu at (309.9, 229.0)
- added C233: 100nF, Capacitor_SMD:C_0402_1005Metric, B.Cu at (298.4, 233.0)
- added C234: 100nF, Capacitor_SMD:C_0402_1005Metric, B.Cu at (292.6, 225.1)
- added C235: 100nF, Capacitor_SMD:C_0402_1005Metric, B.Cu at (301.3, 231.0)
- added C236: 100nF, Capacitor_SMD:C_0402_1005Metric, B.Cu at (304.1, 229.0)
- added C237: 100nF, Capacitor_SMD:C_0402_1005Metric, B.Cu at (298.4, 223.1)
- added C238: 100nF, Capacitor_SMD:C_0402_1005Metric, B.Cu at (298.4, 229.0)
- added C239: 100nF, Capacitor_SMD:C_0402_1005Metric, B.Cu at (292.6, 223.1)
- added C240: 100nF, Capacitor_SMD:C_0402_1005Metric, B.Cu at (298.4, 225.1)
- added C241: 100nF, Capacitor_SMD:C_0402_1005Metric, B.Cu at (307.0, 223.1)
- added C242: 100nF, Capacitor_SMD:C_0402_1005Metric, B.Cu at (295.5, 229.0)
- added C243: 100nF, Capacitor_SMD:C_0402_1005Metric, B.Cu at (309.9, 233.0)
- added C244: 100nF, Capacitor_SMD:C_0402_1005Metric, B.Cu at (295.5, 223.1)
- added C245: 100nF, Capacitor_SMD:C_0402_1005Metric, B.Cu at (301.3, 227.1)
- added C246: 100nF, Capacitor_SMD:C_0402_1005Metric, B.Cu at (304.1, 223.1)
- added C247: 100nF, Capacitor_SMD:C_0402_1005Metric, B.Cu at (304.1, 233.0)
- added C301: 22pF, Capacitor_SMD:C_0402_1005Metric, B.Cu at (423.7, 361.5)
- added C302: 22pF, Capacitor_SMD:C_0402_1005Metric, B.Cu at (382.1, 319.2)
- added C303: 1uF, Capacitor_SMD:C_0402_1005Metric, B.Cu at (408.4, 345.1)
- added C304: .1uF, Capacitor_SMD:C_0402_1005Metric, B.Cu at (440.9, 378.4)
- added C305: .1uF, Capacitor_SMD:C_0402_1005Metric, B.Cu at (402.9, 339.9)
- added C306: .1uF, Capacitor_SMD:C_0402_1005Metric, B.Cu at (385.0, 322.6)
- added C307: 10uf, Capacitor_SMD:C_0402_1005Metric, B.Cu at (354.0, 291.4)
- added C308: 100nF, Capacitor_SMD:C_0402_1005Metric, B.Cu at (174.6, 253.1)
- added C309: 100nF, Capacitor_SMD:C_0402_1005Metric, B.Cu at (183.2, 263.0)
- added C310: 100nF, Capacitor_SMD:C_0402_1005Metric, B.Cu at (180.4, 259.0)
- added C311: 100nF, Capacitor_SMD:C_0402_1005Metric, B.Cu at (191.9, 253.1)
- added C312: 100nF, Capacitor_SMD:C_0402_1005Metric, B.Cu at (177.5, 255.1)
- added C313: 100nF, Capacitor_SMD:C_0402_1005Metric, B.Cu at (186.1, 263.0)
- added C314: 100nF, Capacitor_SMD:C_0402_1005Metric, B.Cu at (186.1, 253.1)
- added C315: 100nF, Capacitor_SMD:C_0402_1005Metric, B.Cu at (189.0, 253.1)
- added C316: 100nF, Capacitor_SMD:C_0402_1005Metric, B.Cu at (180.4, 253.1)
- added C317: 100nF, Capacitor_SMD:C_0402_1005Metric, B.Cu at (174.6, 255.1)
- added C318: 100nF, Capacitor_SMD:C_0402_1005Metric, B.Cu at (191.9, 257.1)
- added C319: 100nF, Capacitor_SMD:C_0402_1005Metric, B.Cu at (191.9, 261.0)
- added C320: 100nF, Capacitor_SMD:C_0402_1005Metric, B.Cu at (183.2, 261.0)
- added C321: 100nF, Capacitor_SMD:C_0402_1005Metric, B.Cu at (183.2, 253.1)
- added C322: 100nF, Capacitor_SMD:C_0402_1005Metric, B.Cu at (177.5, 257.1)
- added C323: 100nF, Capacitor_SMD:C_0402_1005Metric, B.Cu at (186.1, 259.0)
- added C324: 100nF, Capacitor_SMD:C_0402_1005Metric, B.Cu at (189.0, 255.1)
- added C325: 100nF, Capacitor_SMD:C_0402_1005Metric, B.Cu at (194.7, 253.1)
- added C326: 100nF, Capacitor_SMD:C_0402_1005Metric, B.Cu at (194.7, 255.1)
- added C327: 100nF, Capacitor_SMD:C_0402_1005Metric, B.Cu at (194.7, 257.1)
- added C328: 100nF, Capacitor_SMD:C_0402_1005Metric, B.Cu at (186.1, 257.1)
- added C329: 100nF, Capacitor_SMD:C_0402_1005Metric, B.Cu at (191.9, 255.1)
- added C330: 100nF, Capacitor_SMD:C_0402_1005Metric, B.Cu at (191.9, 263.0)
- added C331: 100nF, Capacitor_SMD:C_0402_1005Metric, B.Cu at (194.7, 259.0)
- added C332: 100nF, Capacitor_SMD:C_0402_1005Metric, B.Cu at (177.5, 259.0)
- added C333: 100nF, Capacitor_SMD:C_0402_1005Metric, B.Cu at (189.0, 257.1)
- added C334: 100nF, Capacitor_SMD:C_0402_1005Metric, B.Cu at (189.0, 259.0)
- added C335: 100nF, Capacitor_SMD:C_0402_1005Metric, B.Cu at (180.4, 261.0)
- added C336: 100nF, Capacitor_SMD:C_0402_1005Metric, B.Cu at (183.2, 259.0)
- added C337: 100nF, Capacitor_SMD:C_0402_1005Metric, B.Cu at (194.7, 263.0)
- added C338: 100nF, Capacitor_SMD:C_0402_1005Metric, B.Cu at (194.7, 261.0)
- added C339: 100nF, Capacitor_SMD:C_0402_1005Metric, B.Cu at (186.1, 261.0)
- added C340: 100nF, Capacitor_SMD:C_0402_1005Metric, B.Cu at (189.0, 261.0)
- added C341: 100nF, Capacitor_SMD:C_0402_1005Metric, B.Cu at (186.1, 255.1)
- added C342: 100nF, Capacitor_SMD:C_0402_1005Metric, B.Cu at (180.4, 257.1)
- added C343: 100nF, Capacitor_SMD:C_0402_1005Metric, B.Cu at (177.5, 253.1)
- added C344: 100nF, Capacitor_SMD:C_0402_1005Metric, B.Cu at (180.4, 255.1)
- added C345: 100nF, Capacitor_SMD:C_0402_1005Metric, B.Cu at (189.0, 263.0)
- added C346: 100nF, Capacitor_SMD:C_0402_1005Metric, B.Cu at (183.2, 255.1)
- added C347: 100nF, Capacitor_SMD:C_0402_1005Metric, B.Cu at (191.9, 259.0)
- added C348: 100nF, Capacitor_SMD:C_0402_1005Metric, B.Cu at (183.2, 257.1)
- added D201: PRTR5V0U2X, Package_TO_SOT_SMD:SOT-143, B.Cu at (59.0, 83.3)
- added D202: PRTR5V0U2X, Package_TO_SOT_SMD:SOT-143, B.Cu at (-75.5, 122.0)
- added D203: NeoPixel_THT, kicad-keyboard-parts.pretty:LED_RGB_Wuerth-PLCC4_3.2x2.8mm_150141M173100, B.Cu at (-18.5, 104.0)
- added D204: NeoPixel_THT, kicad-keyboard-parts.pretty:LED_RGB_Wuerth-PLCC4_3.2x2.8mm_150141M173100, B.Cu at (-27.5, 105.0)
- added D205: NeoPixel_THT, kicad-keyboard-parts.pretty:LED_RGB_Wuerth-PLCC4_3.2x2.8mm_150141M173100, B.Cu at (-36.5, 104.0)
- added D206: NeoPixel_THT, kicad-keyboard-parts.pretty:LED_RGB_Wuerth-PLCC4_3.2x2.8mm_150141M173100, B.Cu at (-45.5, 105.0)
- added D207: NeoPixel_THT, kicad-keyboard-parts.pretty:LED_RGB_Wuerth-PLCC4_3.2x2.8mm_150141M173100, B.Cu at (-55.5, 91.0)
- added D208: NeoPixel_THT, kicad-keyboard-parts.pretty:LED_RGB_Wuerth-PLCC4_3.2x2.8mm_150141M173100, B.Cu at (-64.5, 90.0)
- added D209: NeoPixel_THT, kicad-keyboard-parts.pretty:LED_RGB_Wuerth-PLCC4_3.2x2.8mm_150141M173100, B.Cu at (-54.5, 104.0)
- added D210: NeoPixel_THT, kicad-keyboard-parts.pretty:LED_RGB_Wuerth-PLCC4_3.2x2.8mm_150141M173100, B.Cu at (-63.5, 105.0)
- added D211: NeoPixel_THT, kicad-keyboard-parts.pretty:LED_RGB_Wuerth-PLCC4_3.2x2.8mm_150141M173100, B.Cu at (-72.5, 103.0)
- added D212: NeoPixel_THT, kicad-keyboard-parts.pretty:LED_RGB_Wuerth-PLCC4_3.2x2.8mm_150141M173100, B.Cu at (-73.5, 91.0)
- added D213: NeoPixel_THT, kicad-keyboard-parts.pretty:LED_RGB_Wuerth-PLCC4_3.2x2.8mm_150141M173100, B.Cu at (-45.5, 86.0)
- added D214: NeoPixel_THT, kicad-keyboard-parts.pretty:LED_RGB_Wuerth-PLCC4_3.2x2.8mm_150141M173100, B.Cu at (-54.5, 85.0)
- added D215: NeoPixel_THT, kicad-keyboard-parts.pretty:LED_RGB_Wuerth-PLCC4_3.2x2.8mm_150141M173100, B.Cu at (-83.5, 126.0)
- added D216: NeoPixel_THT, kicad-keyboard-parts.pretty:LED_RGB_Wuerth-PLCC4_3.2x2.8mm_150141M173100, B.Cu at (-123.5, 122.0)
- added D217: NeoPixel_THT, kicad-keyboard-parts.pretty:LED_RGB_Wuerth-PLCC4_3.2x2.8mm_150141M173100, B.Cu at (-126.5, 89.0)
- added D218: NeoPixel_THT, kicad-keyboard-parts.pretty:LED_RGB_Wuerth-PLCC4_3.2x2.8mm_150141M173100, B.Cu at (-128.5, 105.0)
- added D219: NeoPixel_THT, kicad-keyboard-parts.pretty:LED_RGB_Wuerth-PLCC4_3.2x2.8mm_150141M173100, B.Cu at (-137.5, 89.0)
- added D220: NeoPixel_THT, kicad-keyboard-parts.pretty:LED_RGB_Wuerth-PLCC4_3.2x2.8mm_150141M173100, B.Cu at (-91.5, 91.0)
- added D221: NeoPixel_THT, kicad-keyboard-parts.pretty:LED_RGB_Wuerth-PLCC4_3.2x2.8mm_150141M173100, B.Cu at (-76.5, 85.0)
- added D222: NeoPixel_THT, kicad-keyboard-parts.pretty:LED_RGB_Wuerth-PLCC4_3.2x2.8mm_150141M173100, B.Cu at (-18.5, 81.0)
- added D223: NeoPixel_THT, kicad-keyboard-parts.pretty:LED_RGB_Wuerth-PLCC4_3.2x2.8mm_150141M173100, B.Cu at (-54.5, 79.0)
- added D224: NeoPixel_THT, kicad-keyboard-parts.pretty:LED_RGB_Wuerth-PLCC4_3.2x2.8mm_150141M173100, B.Cu at (-76.5, 79.0)
- added D225: NeoPixel_THT, kicad-keyboard-parts.pretty:LED_RGB_Wuerth-PLCC4_3.2x2.8mm_150141M173100, B.Cu at (-81.5, 105.0)
- added D226: NeoPixel_THT, kicad-keyboard-parts.pretty:LED_RGB_Wuerth-PLCC4_3.2x2.8mm_150141M173100, B.Cu at (-137.5, 95.0)
- added D227: NeoPixel_THT, kicad-keyboard-parts.pretty:LED_RGB_Wuerth-PLCC4_3.2x2.8mm_150141M173100, B.Cu at (-115.5, 99.0)
- added D228: NeoPixel_THT, kicad-keyboard-parts.pretty:LED_RGB_Wuerth-PLCC4_3.2x2.8mm_150141M173100, B.Cu at (-105.5, 105.0)
- added D229: NeoPixel_THT, kicad-keyboard-parts.pretty:LED_RGB_Wuerth-PLCC4_3.2x2.8mm_150141M173100, B.Cu at (-137.5, 101.0)
- added D230: NeoPixel_THT, kicad-keyboard-parts.pretty:LED_RGB_Wuerth-PLCC4_3.2x2.8mm_150141M173100, B.Cu at (-84.5, 111.0)
- added D231: NeoPixel_THT, kicad-keyboard-parts.pretty:LED_RGB_Wuerth-PLCC4_3.2x2.8mm_150141M173100, B.Cu at (-63.5, 84.0)
- added D232: NeoPixel_THT, kicad-keyboard-parts.pretty:LED_RGB_Wuerth-PLCC4_3.2x2.8mm_150141M173100, B.Cu at (-83.5, 120.0)
- added D233: NeoPixel_THT, kicad-keyboard-parts.pretty:LED_RGB_Wuerth-PLCC4_3.2x2.8mm_150141M173100, B.Cu at (-141.5, 107.0)
- added D234: NeoPixel_THT, kicad-keyboard-parts.pretty:LED_RGB_Wuerth-PLCC4_3.2x2.8mm_150141M173100, B.Cu at (-94.5, 122.0)
- added D235: NeoPixel_THT, kicad-keyboard-parts.pretty:LED_RGB_Wuerth-PLCC4_3.2x2.8mm_150141M173100, B.Cu at (-96.5, 105.0)
- added D236: NeoPixel_THT, kicad-keyboard-parts.pretty:LED_RGB_Wuerth-PLCC4_3.2x2.8mm_150141M173100, B.Cu at (-147.5, 85.0)
- added D237: NeoPixel_THT, kicad-keyboard-parts.pretty:LED_RGB_Wuerth-PLCC4_3.2x2.8mm_150141M173100, B.Cu at (-142.5, 122.0)
- added D238: NeoPixel_THT, kicad-keyboard-parts.pretty:LED_RGB_Wuerth-PLCC4_3.2x2.8mm_150141M173100, B.Cu at (-26.5, 87.0)
- added D239: NeoPixel_THT, kicad-keyboard-parts.pretty:LED_RGB_Wuerth-PLCC4_3.2x2.8mm_150141M173100, B.Cu at (-35.5, 87.0)
- added D240: NeoPixel_THT, kicad-keyboard-parts.pretty:LED_RGB_Wuerth-PLCC4_3.2x2.8mm_150141M173100, B.Cu at (-36.5, 81.0)
- added D241: NeoPixel_THT, kicad-keyboard-parts.pretty:LED_RGB_Wuerth-PLCC4_3.2x2.8mm_150141M173100, B.Cu at (-45.5, 80.0)
- added D242: NeoPixel_THT, kicad-keyboard-parts.pretty:LED_RGB_Wuerth-PLCC4_3.2x2.8mm_150141M173100, B.Cu at (-27.5, 81.0)
- added D243: D_Small, Diode_SMD:D_SOD-123, B.Cu at (-136.5, 138.0)
- added D244: D_Small, Diode_SMD:D_SOD-123, B.Cu at (-129.5, 136.0)
- added D245: D_Small, Diode_SMD:D_SOD-123, B.Cu at (-120.5, 105.0)
- added D246: D_Small, Diode_SMD:D_SOD-123, B.Cu at (-105.5, 159.0)
- added D247: D_Small, Diode_SMD:D_SOD-123, B.Cu at (-81.5, 91.0)
- added D248: D_Small, Diode_SMD:D_SOD-123, B.Cu at (-104.5, 129.0)
- added D249: D_Small, Diode_SMD:D_SOD-123, B.Cu at (-122.5, 138.0)
- added D250: D_Small, Diode_SMD:D_SOD-123, B.Cu at (-114.5, 94.0)
- added D251: D_Small, Diode_SMD:D_SOD-123, B.Cu at (-115.5, 160.0)
- added D252: D_Small, Diode_SMD:D_SOD-123, B.Cu at (-78.5, 97.0)
- added D253: D_Small, Diode_SMD:D_SOD-123, B.Cu at (-102.5, 119.0)
- added D254: D_Small, Diode_SMD:D_SOD-123, B.Cu at (-110.5, 136.0)
- added D255: D_Small, Diode_SMD:D_SOD-123, B.Cu at (-52.5, 143.0)
- added D256: D_Small, Diode_SMD:D_SOD-123, B.Cu at (-96.5, 153.0)
- added D257: D_Small, Diode_SMD:D_SOD-123, B.Cu at (-61.5, 97.0)
- added D258: D_Small, Diode_SMD:D_SOD-123, B.Cu at (-69.5, 114.0)
- added D259: D_Small, Diode_SMD:D_SOD-123, B.Cu at (-82.5, 135.0)
- added D260: D_Small, Diode_SMD:D_SOD-123, B.Cu at (-53.5, 153.0)
- added D261: D_Small, Diode_SMD:D_SOD-123, B.Cu at (-74.5, 156.0)
- added D262: LED, LED_SMD:LED_PLCC_2835, B.Cu at (-10.5, 80.0)
- added D263: D_Small, Diode_SMD:D_SOD-123, B.Cu at (-45.5, 91.0)
- added D264: D_Small, Diode_SMD:D_SOD-123, B.Cu at (-60.5, 120.0)
- added D265: D_Small, Diode_SMD:D_SOD-123, B.Cu at (-62.5, 136.0)
- added D266: D_Small, Diode_SMD:D_SOD-123, B.Cu at (-47.5, 111.0)
- added D267: D_Small, Diode_SMD:D_SOD-123, B.Cu at (-50.5, 172.0)
- added D268: D_Small, Diode_SMD:D_SOD-123, B.Cu at (-43.5, 97.0)
- added D269: D_Small, Diode_SMD:D_SOD-123, B.Cu at (-66.5, 119.0)
- added D270: D_Small, Diode_SMD:D_SOD-123, B.Cu at (-104.5, 136.0)
- added D271: D_Small, Diode_SMD:D_SOD-123, B.Cu at (-17.5, 153.0)
- added D272: D_Small, Diode_SMD:D_SOD-123, B.Cu at (-103.5, 149.0)
- added D273: D_Small, Diode_SMD:D_SOD-123, B.Cu at (-7.53, 97.0)
- added D274: D_Small, Diode_SMD:D_SOD-123, B.Cu at (-24.5, 120.0)
- added D275: D_Small, Diode_SMD:D_SOD-123, B.Cu at (-56.5, 136.0)
- added D276: D_Small, Diode_SMD:D_SOD-123, B.Cu at (-34.5, 143.0)
- added D277: D_Small, Diode_SMD:D_SOD-123, B.Cu at (-55.5, 159.0)
- added D278: D_Small, Diode_SMD:D_SOD-123, B.Cu at (-25.5, 97.0)
- added D279: D_Small, Diode_SMD:D_SOD-123, B.Cu at (-30.5, 119.0)
- added D280: D_Small, Diode_SMD:D_SOD-123, B.Cu at (-116.5, 136.0)
- added D281: D_Small, Diode_SMD:D_SOD-123, B.Cu at (-16.5, 143.0)
- added D282: D_Small, Diode_SMD:D_SOD-123, B.Cu at (-97.5, 97.0)
- added D301: PRTR5V0U2X, Package_TO_SOT_SMD:SOT-143, B.Cu at (381.2, 314.1)
- added D302: PRTR5V0U2X, Package_TO_SOT_SMD:SOT-143, B.Cu at (355.6, 87.0)
- added D303: NeoPixel_THT, kicad-keyboard-parts.pretty:LED_RGB_Wuerth-PLCC4_3.2x2.8mm_150141M173100, B.Cu at (374.8, 305.3)
- added D304: NeoPixel_THT, kicad-keyboard-parts.pretty:LED_RGB_Wuerth-PLCC4_3.2x2.8mm_150141M173100, B.Cu at (412.6, 344.4)
- added D305: NeoPixel_THT, kicad-keyboard-parts.pretty:LED_RGB_Wuerth-PLCC4_3.2x2.8mm_150141M173100, B.Cu at (407.1, 340.0)
- added D306: NeoPixel_THT, kicad-keyboard-parts.pretty:LED_RGB_Wuerth-PLCC4_3.2x2.8mm_150141M173100, B.Cu at (407.8, 335.6)
- added D307: NeoPixel_THT, kicad-keyboard-parts.pretty:LED_RGB_Wuerth-PLCC4_3.2x2.8mm_150141M173100, B.Cu at (436.3, 366.0)
- added D308: NeoPixel_THT, kicad-keyboard-parts.pretty:LED_RGB_Wuerth-PLCC4_3.2x2.8mm_150141M173100, B.Cu at (456.5, 379.5)
- added D309: NeoPixel_THT, kicad-keyboard-parts.pretty:LED_RGB_Wuerth-PLCC4_3.2x2.8mm_150141M173100, B.Cu at (400.0, 321.7)
- added D310: NeoPixel_THT, kicad-keyboard-parts.pretty:LED_RGB_Wuerth-PLCC4_3.2x2.8mm_150141M173100, B.Cu at (358.0, 280.8)
- added D311: NeoPixel_THT, kicad-keyboard-parts.pretty:LED_RGB_Wuerth-PLCC4_3.2x2.8mm_150141M173100, B.Cu at (346.5, 274.1)
- added D312: NeoPixel_THT, kicad-keyboard-parts.pretty:LED_RGB_Wuerth-PLCC4_3.2x2.8mm_150141M173100, B.Cu at (358.0, 285.1)
- added D313: NeoPixel_THT, kicad-keyboard-parts.pretty:LED_RGB_Wuerth-PLCC4_3.2x2.8mm_150141M173100, B.Cu at (380.3, 305.3)
- added D314: NeoPixel_THT, kicad-keyboard-parts.pretty:LED_RGB_Wuerth-PLCC4_3.2x2.8mm_150141M173100, B.Cu at (402.2, 334.8)
- added D315: NeoPixel_THT, kicad-keyboard-parts.pretty:LED_RGB_Wuerth-PLCC4_3.2x2.8mm_150141M173100, B.Cu at (407.8, 331.3)
- added D316: NeoPixel_THT, kicad-keyboard-parts.pretty:LED_RGB_Wuerth-PLCC4_3.2x2.8mm_150141M173100, B.Cu at (380.3, 309.6)
- added D317: NeoPixel_THT, kicad-keyboard-parts.pretty:LED_RGB_Wuerth-PLCC4_3.2x2.8mm_150141M173100, B.Cu at (436.3, 361.6)
- added D318: NeoPixel_THT, kicad-keyboard-parts.pretty:LED_RGB_Wuerth-PLCC4_3.2x2.8mm_150141M173100, B.Cu at (402.0, 330.4)
- added D319: NeoPixel_THT, kicad-keyboard-parts.pretty:LED_RGB_Wuerth-PLCC4_3.2x2.8mm_150141M173100, B.Cu at (402.0, 326.1)
- added D320: NeoPixel_THT, kicad-keyboard-parts.pretty:LED_RGB_Wuerth-PLCC4_3.2x2.8mm_150141M173100, B.Cu at (364.6, 291.8)
- added D321: NeoPixel_THT, kicad-keyboard-parts.pretty:LED_RGB_Wuerth-PLCC4_3.2x2.8mm_150141M173100, B.Cu at (418.2, 341.9)
- added D322: NeoPixel_THT, kicad-keyboard-parts.pretty:LED_RGB_Wuerth-PLCC4_3.2x2.8mm_150141M173100, B.Cu at (430.8, 362.6)
- added D323: NeoPixel_THT, kicad-keyboard-parts.pretty:LED_RGB_Wuerth-PLCC4_3.2x2.8mm_150141M173100, B.Cu at (346.7, 278.4)
- added D324: NeoPixel_THT, kicad-keyboard-parts.pretty:LED_RGB_Wuerth-PLCC4_3.2x2.8mm_150141M173100, B.Cu at (425.0, 358.3)
- added D325: NeoPixel_THT, kicad-keyboard-parts.pretty:LED_RGB_Wuerth-PLCC4_3.2x2.8mm_150141M173100, B.Cu at (394.5, 321.7)
- added D326: NeoPixel_THT, kicad-keyboard-parts.pretty:LED_RGB_Wuerth-PLCC4_3.2x2.8mm_150141M173100, B.Cu at (418.2, 346.3)
- added D327: NeoPixel_THT, kicad-keyboard-parts.pretty:LED_RGB_Wuerth-PLCC4_3.2x2.8mm_150141M173100, B.Cu at (418.2, 350.6)
- added D328: NeoPixel_THT, kicad-keyboard-parts.pretty:LED_RGB_Wuerth-PLCC4_3.2x2.8mm_150141M173100, B.Cu at (352.4, 281.8)
- added D329: NeoPixel_THT, kicad-keyboard-parts.pretty:LED_RGB_Wuerth-PLCC4_3.2x2.8mm_150141M173100, B.Cu at (386.1, 311.1)
- added D330: NeoPixel_THT, kicad-keyboard-parts.pretty:LED_RGB_Wuerth-PLCC4_3.2x2.8mm_150141M173100, B.Cu at (352.2, 277.4)
- added D331: NeoPixel_THT, kicad-keyboard-parts.pretty:LED_RGB_Wuerth-PLCC4_3.2x2.8mm_150141M173100, B.Cu at (340.9, 274.1)
- added D332: NeoPixel_THT, kicad-keyboard-parts.pretty:LED_RGB_Wuerth-PLCC4_3.2x2.8mm_150141M173100, B.Cu at (396.5, 326.1)
- added D333: NeoPixel_THT, kicad-keyboard-parts.pretty:LED_RGB_Wuerth-PLCC4_3.2x2.8mm_150141M173100, B.Cu at (370.4, 294.2)
- added D334: NeoPixel_THT, kicad-keyboard-parts.pretty:LED_RGB_Wuerth-PLCC4_3.2x2.8mm_150141M173100, B.Cu at (412.6, 340.0)
- added D335: NeoPixel_THT, kicad-keyboard-parts.pretty:LED_RGB_Wuerth-PLCC4_3.2x2.8mm_150141M173100, B.Cu at (363.7, 287.4)
- added D336: NeoPixel_THT, kicad-keyboard-parts.pretty:LED_RGB_Wuerth-PLCC4_3.2x2.8mm_150141M173100, B.Cu at (447.2, 375.1)
- added D337: NeoPixel_THT, kicad-keyboard-parts.pretty:LED_RGB_Wuerth-PLCC4_3.2x2.8mm_150141M173100, B.Cu at (452.7, 375.1)
- added D338: NeoPixel_THT, kicad-keyboard-parts.pretty:LED_RGB_Wuerth-PLCC4_3.2x2.8mm_150141M173100, B.Cu at (451.0, 379.5)
- added D339: NeoPixel_THT, kicad-keyboard-parts.pretty:LED_RGB_Wuerth-PLCC4_3.2x2.8mm_150141M173100, B.Cu at (364.8, 296.1)
- added D340: NeoPixel_THT, kicad-keyboard-parts.pretty:LED_RGB_Wuerth-PLCC4_3.2x2.8mm_150141M173100, B.Cu at (430.6, 358.3)
- added D341: NeoPixel_THT, kicad-keyboard-parts.pretty:LED_RGB_Wuerth-PLCC4_3.2x2.8mm_150141M173100, B.Cu at (386.1, 315.4)
- added D342: NeoPixel_THT, kicad-keyboard-parts.pretty:LED_RGB_Wuerth-PLCC4_3.2x2.8mm_150141M173100, B.Cu at (358.2, 289.4)
- added D343: NeoPixel_THT, kicad-keyboard-parts.pretty:LED_RGB_Wuerth-PLCC4_3.2x2.8mm_150141M173100, B.Cu at (370.4, 298.6)
- added D344: D_Small, Diode_SMD:D_SOD-123, B.Cu at (462.2, 378.0)
- added D345: D_Small, Diode_SMD:D_SOD-123, B.Cu at (464.1, 374.6)
- added D346: D_Small, Diode_SMD:D_SOD-123, B.Cu at (487.1, 378.0)
- added D347: D_Small, Diode_SMD:D_SOD-123, B.Cu at (407.7, 327.4)
- added D348: D_Small, Diode_SMD:D_SOD-123, B.Cu at (467.9, 378.0)
- added D349: D_Small, Diode_SMD:D_SOD-123, B.Cu at (475.6, 374.6)
- added D350: D_Small, Diode_SMD:D_SOD-123, B.Cu at (363.6, 276.9)
- added D351: D_Small, Diode_SMD:D_SOD-123, B.Cu at (407.7, 324.1)
- added D352: D_Small, Diode_SMD:D_SOD-123, B.Cu at (473.7, 378.0)
- added D353: D_Small, Diode_SMD:D_SOD-123, B.Cu at (467.9, 381.4)
- added D354: D_Small, Diode_SMD:D_SOD-123, B.Cu at (376.0, 290.4)
- added D355: D_Small, Diode_SMD:D_SOD-123, B.Cu at (473.7, 381.4)
- added D356: D_Small, Diode_SMD:D_SOD-123, B.Cu at (363.6, 280.2)
- added D357: D_Small, Diode_SMD:D_SOD-123, B.Cu at (363.6, 273.6)
- added D358: D_Small, Diode_SMD:D_SOD-123, B.Cu at (413.4, 334.1)
- added D359: D_Small, Diode_SMD:D_SOD-123, B.Cu at (496.7, 381.4)
- added D360: D_Small, Diode_SMD:D_SOD-123, B.Cu at (485.2, 381.4)
- added D361: D_Small, Diode_SMD:D_SOD-123, B.Cu at (458.4, 374.6)
- added D362: D_Small, Diode_SMD:D_SOD-123, B.Cu at (462.2, 381.4)
- added D363: D_Small, Diode_SMD:D_SOD-123, B.Cu at (363.6, 283.6)
- added D364: LED, LED_SMD:LED_PLCC_2835, B.Cu at (376.1, 300.9)
- added D365: D_Small, Diode_SMD:D_SOD-123, B.Cu at (436.2, 357.8)
- added D366: D_Small, Diode_SMD:D_SOD-123, B.Cu at (381.8, 293.8)
- added D367: D_Small, Diode_SMD:D_SOD-123, B.Cu at (481.4, 374.6)
- added D368: D_Small, Diode_SMD:D_SOD-123, B.Cu at (376.0, 293.8)
- added D369: D_Small, Diode_SMD:D_SOD-123, B.Cu at (357.9, 276.9)
- added D370: D_Small, Diode_SMD:D_SOD-123, B.Cu at (381.8, 290.4)
- added D371: D_Small, Diode_SMD:D_SOD-123, B.Cu at (370.3, 290.4)
- added D372: D_Small, Diode_SMD:D_SOD-123, B.Cu at (487.1, 374.6)
- added D373: D_Small, Diode_SMD:D_SOD-123, B.Cu at (420.8, 324.8)
- added D374: D_Small, Diode_SMD:D_SOD-123, B.Cu at (479.4, 381.4)
- added D375: D_Small, Diode_SMD:D_SOD-123, B.Cu at (357.9, 273.6)
- added D376: D_Small, Diode_SMD:D_SOD-123, B.Cu at (413.4, 324.1)
- added D377: D_Small, Diode_SMD:D_SOD-123, B.Cu at (413.4, 327.4)
- added D378: D_Small, Diode_SMD:D_SOD-123, B.Cu at (413.4, 330.8)
- added D379: D_Small, Diode_SMD:D_SOD-123, B.Cu at (352.1, 273.6)
- added D380: D_Small, Diode_SMD:D_SOD-123, B.Cu at (381.8, 300.4)
- added D381: D_Small, Diode_SMD:D_SOD-123, B.Cu at (490.9, 381.4)
- added D382: D_Small, Diode_SMD:D_SOD-123, B.Cu at (381.8, 297.1)
- added D383: D_Small, Diode_SMD:D_SOD-123, B.Cu at (479.4, 378.0)
- added D384: D_Small, Diode_SMD:D_SOD-123, B.Cu at (469.9, 374.6)
- added D385: D_Small, Diode_SMD:D_SOD-123, B.Cu at (376.0, 297.1)
- added F201: 500m, Keebio-Parts:Fuse_0805, B.Cu at (60.0, 79.0)
- added F301: 500m, Keebio-Parts:Fuse_0805, B.Cu at (346.8, 77.8)
- added FB201: FerriteBead_Small, Inductor_SMD:L_0805_2012Metric_Pad1.15x1.40mm_HandSolder, B.Cu at (40.5, 79.5)
- added FB301: FerriteBead_Small, Inductor_SMD:L_0805_2012Metric_Pad1.15x1.40mm_HandSolder, B.Cu at (365.0, 79.2)
- added H201: MountingHole, MountingHole:MountingHole_2.2mm_M2_DIN965_Pad, F.Cu at (34.0, 79.0)
- added H202: MountingHole, MountingHole:MountingHole_2.2mm_M2_DIN965_Pad, F.Cu at (114.0, 79.0)
- added H203: MountingHole, MountingHole:MountingHole_2.2mm_M2_DIN965_Pad, F.Cu at (194.0, 79.0)
- added H204: MountingHole, MountingHole:MountingHole_2.2mm_M2_DIN965_Pad, F.Cu at (34.0, 171.0)
- added H205: MountingHole, MountingHole:MountingHole_2.2mm_M2_DIN965_Pad, F.Cu at (116.2, 171.0)
- added H206: MountingHole, MountingHole:MountingHole_2.2mm_M2_DIN965_Pad, F.Cu at (198.5, 171.0)
- added H301: MountingHole, MountingHole:MountingHole_2.2mm_M2_DIN965_Pad, F.Cu at (215.5, 79.0)
- added H302: MountingHole, MountingHole:MountingHole_2.2mm_M2_DIN965_Pad, F.Cu at (293.2, 79.0)
- added H303: MountingHole, MountingHole:MountingHole_2.2mm_M2_DIN965_Pad, F.Cu at (371.0, 79.0)
- added H304: MountingHole, MountingHole:MountingHole_2.2mm_M2_DIN965_Pad, F.Cu at (220.0, 171.0)
- added H305: MountingHole, MountingHole:MountingHole_2.2mm_M2_DIN965_Pad, F.Cu at (295.5, 171.0)
- added H306: MountingHole, MountingHole:MountingHole_2.2mm_M2_DIN965_Pad, F.Cu at (371.0, 171.0)
- added J201: USB_C_Receptacle_USB2.0, Type-C:HRO-TYPE-C-31-M-13, B.Cu at (49.5, 75.0)
- added J202: USB_C_Receptacle_USB2.0, Type-C:HRO-TYPE-C-31-M-13, B.Cu at (-90.5, 86.0)
- added J203: AVR-ISP-6, Keebio-Parts:ICSP-Header, B.Cu at (137.7, 80.0)
- added J301: USB_C_Receptacle_USB2.0, Type-C:HRO-TYPE-C-31-M-13, B.Cu at (507.1, 381.6)
- added J302: USB_C_Receptacle_USB2.0, Type-C:HRO-TYPE-C-31-M-13, B.Cu at (355.5, 75.0)
- added J303: AVR-ISP-6, Keebio-Parts:ICSP-Header, B.Cu at (271.9, 80.0)
- added Q202: DMN2041L, Package_TO_SOT_SMD:SOT-23, B.Cu at (-105.5, 124.0)
- added Q302: DMN2041L, Package_TO_SOT_SMD:SOT-23, B.Cu at (352.8, 286.1)
- added R201: 5.1k, Resistor_SMD:R_0402_1005Metric, B.Cu at (-127.5, 93.0)
- added R202: 5.1k, Resistor_SMD:R_0402_1005Metric, B.Cu at (-92.5, 95.0)
- added R203: 5.1k, Resistor_SMD:R_0402_1005Metric, B.Cu at (-127.5, 96.0)
- added R204: 5.1k, Resistor_SMD:R_0402_1005Metric, B.Cu at (-88.5, 96.0)
- added R205: 300, Resistor_SMD:R_0402_1005Metric, B.Cu at (-70.5, 96.0)
- added R220: 22, Resistor_SMD:R_0402_1005Metric, B.Cu at (-123.5, 97.0)
- added R224: 22, Resistor_SMD:R_0402_1005Metric, B.Cu at (-129.5, 101.0)
- added R225: 10k, Resistor_SMD:R_0402_1005Metric, B.Cu at (-120.5, 127.0)
- added R238: 10k, Resistor_SMD:R_0402_1005Metric, B.Cu at (-105.5, 93.0)
- added R242: 4.7K, Resistor_SMD:R_0402_1005Metric, B.Cu at (-98.5, 93.0)
- added R243: 4.7K, Resistor_SMD:R_0402_1005Metric, B.Cu at (-84.5, 97.0)
- added R252: 470, Resistor_SMD:R_0402_1005Metric, B.Cu at (-13.5, 97.0)
- added R253: 1k, Resistor_SMD:R_0402_1005Metric, B.Cu at (-106.5, 101.0)
- added R301: 5.1k, Resistor_SMD:R_0402_1005Metric, B.Cu at (432.1, 365.8)
- added R302: 5.1k, Resistor_SMD:R_0402_1005Metric, B.Cu at (358.5, 85.8)
- added R303: 5.1k, Resistor_SMD:R_0402_1005Metric, B.Cu at (381.9, 317.3)
- added R304: 5.1k, Resistor_SMD:R_0402_1005Metric, B.Cu at (352.5, 85.8)
- added R305: 300, Resistor_SMD:R_0402_1005Metric, B.Cu at (392.2, 325.0)
- added R323: 22, Resistor_SMD:R_0402_1005Metric, B.Cu at (317.6, 97.0)
- added R327: 22, Resistor_SMD:R_0402_1005Metric, B.Cu at (316.4, 97.0)
- added R328: 10k, Resistor_SMD:R_0402_1005Metric, B.Cu at (336.7, 272.9)
- added R341: 10k, Resistor_SMD:R_0402_1005Metric, B.Cu at (376.1, 308.5)
- added R345: 4.7K, Resistor_SMD:R_0402_1005Metric, B.Cu at (342.4, 277.2)
- added R346: 4.7K, Resistor_SMD:R_0402_1005Metric, B.Cu at (457.9, 382.7)
- added R353: 470, Resistor_SMD:R_0402_1005Metric, B.Cu at (420.8, 357.1)
- added R354: 1k, Resistor_SMD:R_0402_1005Metric, B.Cu at (402.9, 337.9)
- added SW201: SW_Push, Button_Switch_SMD:SW_SPST_SKQG_WithStem, B.Cu at (145.5, 87.2)
- added SW202: RotaryEncoder, Rotary_Encoder.pretty:kailh_EN97xx_rotary_encoder, F.Cu at (40.5, 93.5)
- added SW203: SW_Push, keyswitches.pretty-2:Kailh_socket_PG1350, F.Cu at (40.5, 110.5)
- added SW204: SW_Push, keyswitches.pretty-2:Kailh_socket_PG1350, F.Cu at (40.5, 127.5)
- added SW205: SW_Push, keyswitches.pretty-2:Kailh_socket_PG1350, F.Cu at (40.5, 144.5)
- added SW206: SW_Push, keyswitches.pretty-2:Kailh_socket_PG1350, F.Cu at (40.5, 161.5)
- added SW207: SW_Push, keyswitches.pretty-2:Kailh_socket_PG1350, F.Cu at (58.5, 93.5)
- added SW208: SW_Push, keyswitches.pretty-2:Kailh_socket_PG1350, F.Cu at (58.5, 110.5)
- added SW209: SW_Push, keyswitches.pretty-2:Kailh_socket_PG1350, F.Cu at (58.5, 127.5)
- added SW210: SW_Push, keyswitches.pretty-2:Kailh_socket_PG1350, F.Cu at (58.5, 144.5)
- added SW211: SW_Push, keyswitches.pretty-2:Kailh_socket_PG1350, F.Cu at (58.5, 161.5)
- added SW212: SW_Push, keyswitches.pretty-2:Kailh_socket_PG1350, F.Cu at (99.0, 93.5)
- added SW213: SW_Push, keyswitches.pretty-2:Kailh_socket_PG1350_1.5U, F.Cu at (85.5, 110.5)
- added SW214: SW_Push, keyswitches.pretty-2:Kailh_socket_PG1350_1.75U, F.Cu at (87.8, 127.5)
- added SW215: SW_Push, keyswitches.pretty-2:Kailh_socket_PG1350_2.25U, F.Cu at (92.2, 144.5)
- added SW216: SW_Push, keyswitches.pretty-2:Kailh_socket_PG1350_1.25U, F.Cu at (83.2, 161.5)
- added SW217: SW_Push, keyswitches.pretty-2:Kailh_socket_PG1350, F.Cu at (117.0, 93.5)
- added SW218: SW_Push, keyswitches.pretty-2:Kailh_socket_PG1350, F.Cu at (108.0, 110.5)
- added SW219: SW_Push, keyswitches.pretty-2:Kailh_socket_PG1350, F.Cu at (112.5, 127.5)
- added SW220: SW_Push, keyswitches.pretty-2:Kailh_socket_PG1350, F.Cu at (121.5, 144.5)
- added SW221: SW_Push, keyswitches.pretty-2:Kailh_socket_PG1350_1.25U, F.Cu at (105.8, 161.5)
- added SW222: SW_Push, keyswitches.pretty-2:Kailh_socket_PG1350, F.Cu at (135.0, 93.5)
- added SW223: SW_Push, keyswitches.pretty-2:Kailh_socket_PG1350, F.Cu at (126.0, 110.5)
- added SW224: SW_Push, keyswitches.pretty-2:Kailh_socket_PG1350, F.Cu at (130.5, 127.5)
- added SW225: SW_Push, keyswitches.pretty-2:Kailh_socket_PG1350, F.Cu at (139.5, 144.5)
- added SW226: SW_Push, keyswitches.pretty-2:Kailh_socket_PG1350_1.25U, F.Cu at (128.2, 161.5)
- added SW227: SW_Push, keyswitches.pretty-2:Kailh_socket_PG1350, F.Cu at (153.0, 93.5)
- added SW228: SW_Push, keyswitches.pretty-2:Kailh_socket_PG1350, F.Cu at (144.0, 110.5)
- added SW229: SW_Push, keyswitches.pretty-2:Kailh_socket_PG1350, F.Cu at (148.5, 127.5)
- added SW230: SW_Push, keyswitches.pretty-2:Kailh_socket_PG1350, F.Cu at (157.5, 144.5)
- added SW231: SW_Push, keyswitches.pretty-2:Kailh_socket_PG1350_1.25U, F.Cu at (150.8, 161.5)
- added SW232: SW_Push, keyswitches.pretty-2:Kailh_socket_PG1350, F.Cu at (171.0, 93.5)
- added SW233: SW_Push, keyswitches.pretty-2:Kailh_socket_PG1350, F.Cu at (162.0, 110.5)
- added SW234: SW_Push, keyswitches.pretty-2:Kailh_socket_PG1350, F.Cu at (166.5, 127.5)
- added SW235: SW_Push, keyswitches.pretty-2:Kailh_socket_PG1350, F.Cu at (175.5, 144.5)
- added SW236: SW_Push, keyswitches.pretty-2:Kailh_socket_PG1350_2.25U, F.Cu at (182.2, 161.5)
- added SW237: SW_Push, keyswitches.pretty-2:Kailh_socket_PG1350, F.Cu at (189.0, 93.5)
- added SW238: SW_Push, keyswitches.pretty-2:Kailh_socket_PG1350, F.Cu at (180.0, 110.5)
- added SW239: SW_Push, keyswitches.pretty-2:Kailh_socket_PG1350, F.Cu at (184.5, 127.5)
- added SW240: SW_Push, keyswitches.pretty-2:Kailh_socket_PG1350, F.Cu at (193.5, 144.5)
- added SW241: SW_Push, keyswitches.pretty-2:Kailh_socket_PG1350, F.Cu at (81.0, 93.5)
- added SW301: SW_Push, Button_Switch_SMD:SW_SPST_SKQG_WithStem, B.Cu at (267.0, 87.5)
- added SW302: SW_Push, keyswitches.pretty-2:Kailh_socket_PG1350, F.Cu at (220.5, 93.5)
- added SW303: SW_Push, keyswitches.pretty-2:Kailh_socket_PG1350, F.Cu at (211.5, 110.5)
- added SW304: SW_Push, keyswitches.pretty-2:Kailh_socket_PG1350, F.Cu at (216.0, 127.5)
- added SW305: SW_Push, keyswitches.pretty-2:Kailh_socket_PG1350, F.Cu at (225.0, 144.5)
- added SW306: SW_Push, keyswitches.pretty-2:Kailh_socket_PG1350, F.Cu at (238.5, 93.5)
- added SW307: SW_Push, keyswitches.pretty-2:Kailh_socket_PG1350, F.Cu at (229.5, 110.5)
- added SW308: SW_Push, keyswitches.pretty-2:Kailh_socket_PG1350, F.Cu at (234.0, 127.5)
- added SW309: SW_Push, keyswitches.pretty-2:Kailh_socket_PG1350, F.Cu at (243.0, 144.5)
- added SW310: SW_Push, keyswitches.pretty-2:Kailh_socket_PG1350_2.25U, F.Cu at (236.2, 161.5)
- added SW311: SW_Push, keyswitches.pretty-2:Kailh_socket_PG1350, F.Cu at (256.5, 93.5)
- added SW312: SW_Push, keyswitches.pretty-2:Kailh_socket_PG1350, F.Cu at (247.5, 110.5)
- added SW313: SW_Push, keyswitches.pretty-2:Kailh_socket_PG1350, F.Cu at (252.0, 127.5)
- added SW314: SW_Push, keyswitches.pretty-2:Kailh_socket_PG1350, F.Cu at (261.0, 144.5)
- added SW315: SW_Push, keyswitches.pretty-2:Kailh_socket_PG1350_1.25U, F.Cu at (267.8, 161.5)
- added SW316: SW_Push, keyswitches.pretty-2:Kailh_socket_PG1350, F.Cu at (274.5, 93.5)
- added SW317: SW_Push, keyswitches.pretty-2:Kailh_socket_PG1350, F.Cu at (265.5, 110.5)
- added SW318: SW_Push, keyswitches.pretty-2:Kailh_socket_PG1350, F.Cu at (270.0, 127.5)
- added SW319: SW_Push, keyswitches.pretty-2:Kailh_socket_PG1350, F.Cu at (279.0, 144.5)
- added SW320: SW_Push, keyswitches.pretty-2:Kailh_socket_PG1350, F.Cu at (288.0, 161.5)
- added SW321: SW_Push, keyswitches.pretty-2:Kailh_socket_PG1350, F.Cu at (292.5, 93.5)
- added SW322: SW_Push, keyswitches.pretty-2:Kailh_socket_PG1350, F.Cu at (283.5, 110.5)
- added SW323: SW_Push, keyswitches.pretty-2:Kailh_socket_PG1350, F.Cu at (288.0, 127.5)
- added SW324: SW_Push, keyswitches.pretty-2:Kailh_socket_PG1350, F.Cu at (297.0, 144.5)
- added SW325: SW_Push, keyswitches.pretty-2:Kailh_socket_PG1350, F.Cu at (306.0, 161.5)
- added SW326: SW_Push, keyswitches.pretty-2:Kailh_socket_PG1350, F.Cu at (310.5, 93.5)
- added SW327: SW_Push, keyswitches.pretty-2:Kailh_socket_PG1350, F.Cu at (301.5, 110.5)
- added SW328: SW_Push, keyswitches.pretty-2:Kailh_socket_PG1350, F.Cu at (306.0, 127.5)
- added SW329: SW_Push, keyswitches.pretty-2:Kailh_socket_PG1350_1.75U, F.Cu at (321.8, 144.5)
- added SW330: SW_Push, keyswitches.pretty-2:Kailh_socket_PG1350, F.Cu at (328.5, 161.5)
- added SW331: SW_Push, keyswitches.pretty-2:Kailh_socket_PG1350, F.Cu at (328.5, 93.5)
- added SW332: SW_Push, keyswitches.pretty-2:Kailh_socket_PG1350, F.Cu at (319.5, 110.5)
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Routing:
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Other:
- board size 369.1 x 95.2 mm -> 345 x 100 mm

Commit message: did some more work on the keyboard, played around with the rotary footprint
Parts:
- SW201, SW301: footprint Button_Switch_SMD:SW_SPST_SKQG_WithStem -> Keebio-Parts:SW_SPST_TL3342
- SW202: footprint Rotary_Encoder.pretty:kailh_EN97xx_rotary_encoder -> Rotary_Encoder.pretty:Kailh_EN65xx_rotary_encoder
- turned SW202 to 0 degrees
- turned SW302 to 180 degrees
- turned SW303 to 180 degrees
- turned SW304 to 180 degrees
- turned SW305 to 180 degrees

Commit message: did some routing
Parts:
- removed U301: ATmega32U4-A, ATmega32U4:ATmega32U4
- D303, D304, D305, D306, D307, D308, D309, D310, D311, D312, D313, D314, D315, D316, D317, D318, D319, D320, D321, D322, D323, D324, D325, D326, D327, D328, D329, D330, D331, D332, D333, D334, D335, D336, D337, D338, D339, D340, D341, D342, D343: moved to F.Cu
- moved D308 317.7 mm to (328.5, 88.8), turned to 0 degrees
- moved D374 316.9 mm to (334.5, 99.5), turned to 90 degrees
- moved C304 310.7 mm to (333.8, 86.8), turned to -90 degrees
- moved C301 306.5 mm to (301.8, 80.2), turned to 0 degrees
- moved D331 305.1 mm to (552.0, 53.8), turned to 0 degrees
- moved D307 304.5 mm to (310.5, 88.8), turned to 0 degrees
- moved D304 299.5 mm to (256.5, 88.8), turned to 0 degrees
- moved D311 297.5 mm to (546.5, 53.8), turned to 0 degrees
- moved D323 297.3 mm to (546.3, 58.1), turned to 0 degrees
- moved D330 289.9 mm to (540.8, 57.1), turned to 0 degrees
- moved D328 289.7 mm to (540.5, 61.5), turned to 0 degrees
- moved D305 284.1 mm to (274.5, 88.8), turned to 0 degrees
- moved D312 282.6 mm to (535.0, 64.8), turned to 0 degrees
- moved D342 282.3 mm to (534.8, 69.2), turned to 0 degrees
- moved D335 275.5 mm to (529.2, 67.2), turned to 0 degrees
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Routing:
- net /Right/COL_1: track 0.00 -> 106.2 mm, vias 0 -> 5
- net /Right/COL_2: track 0.00 -> 106.2 mm, vias 0 -> 5
- net /Right/COL_0: track 0.00 -> 80.7 mm, vias 0 -> 4
- net +5V: track 22.4 -> 82.5 mm, vias 0 -> 6
- net Net-(C302-Pad1): track 0.00 -> 17.9 mm
- net Net-(C301-Pad2): track 0.00 -> 17.2 mm
- net VCC: track 42.3 -> 58.9 mm
- net GND: track 77.0 -> 83.5 mm, vias 5 -> 7
- net Net-(C202-Pad1): track 0.00 -> 4.57 mm
- net Net-(C201-Pad2): track 0.00 -> 1.73 mm
- added copper zone on B.Cu, net Earth
- added copper zone on F.Cu, net Earth
- added copper zone on B.Cu, net GND
- added copper zone on F.Cu, net GND

Commit message: placed some i2cs
Parts:
- removed D202, D301: PRTR5V0U2X, Package_TO_SOT_SMD:SOT-143
- removed D262, D364: LED, LED_SMD:LED_PLCC_2835
- removed Q202, Q302: DMN2041L, Package_TO_SOT_SMD:SOT-23
- removed R202, R204, R301, R303: 5.1k, Resistor_SMD:R_0402_1005Metric
- removed R252, R353: 470, Resistor_SMD:R_0402_1005Metric
- removed R253, R354: 1k, Resistor_SMD:R_0402_1005Metric
- removed R345, R346: 4.7K, Resistor_SMD:R_0402_1005Metric
- added R1: 4.7K, Resistor_SMD:R_0402_1005Metric, B.Cu at (319.7, 57.4)
- added R2: 4.7K, Resistor_SMD:R_0402_1005Metric, B.Cu at (319.7, 59.4)
- added U301: ATmega32U4-A, ATmega32U4:ATmega32U4, B.Cu at (322.2, 84.8)
- J202, J301: value USB_C_Receptacle_USB2.0 -> Conn_01x04_Female; footprint Type-C:HRO-TYPE-C-31-M-13 -> Keebio-Parts:I2C_Breakout
- SW202: footprint Rotary_Encoder.pretty:Kailh_EN65xx_rotary_encoder -> Rotary_Encoder.pretty:kailh_EN97xx_rotary_encoder
- moved J301 365.9 mm to (217.8, 157.7)
- moved J202 300.0 mm to (200.8, 157.7)
Connections:
- R242 pad 1: Net-(R242-Pad1) -> +5V
- R243 pad 1: Net-(R243-Pad1) -> +5V
- U201 pad 20: Net-(R242-Pad1) -> /Left/DATA_1
- U201 pad 21: Net-(R243-Pad1) -> /Left/DATA_2
Routing:
- net GND: track 83.5 -> 116.7 mm

Commit message: did some more routing
Parts:
- moved C303 270.2 mm to (317.2, 90.8), turned to -135 degrees
Connections:
- U301 pad 1: unconnected-(U301-Pad1) -> /Right/COL_6
- U301 pad 12: Net-(R305-Pad1) -> /Right/COL_3
- U301 pad 18: unconnected-(U301-Pad18) -> /Right/COL_2
- U301 pad 19: /Right/COL_8 -> /Right/COL_1
- U301 pad 22: /Right/ROW_0 -> /Right/COL_0
- U301 pad 29: /Right/COL_6 -> unconnected-(U301-Pad29)
- U301 pad 31: /Right/CAPS_LOCK_PWM -> unconnected-(U301-Pad31)
- U301 pad 36: /Right/COL_5 -> unconnected-(U301-Pad36)
- U301 pad 37: /Right/COL_4 -> unconnected-(U301-Pad37)
- U301 pad 38: /Right/COL_3 -> unconnected-(U301-Pad38)
- U301 pad 39: /Right/COL_2 -> unconnected-(U301-Pad39)
- U301 pad 40: /Right/COL_1 -> unconnected-(U301-Pad40)
- U301 pad 41: /Right/COL_0 -> unconnected-(U301-Pad41)
- U301 pad 8: unconnected-(U301-Pad8) -> Net-(R305-Pad1)
Routing:
- net /Right/COL_5: track 0.00 -> 113.7 mm, vias 0 -> 5
- net /Right/COL_3: track 0.00 -> 108.9 mm, vias 0 -> 5
- net /Right/COL_4: track 0.00 -> 108.2 mm, vias 0 -> 5
- net /Right/COL_7: track 0.00 -> 100.1 mm, vias 0 -> 5
- net /Right/COL_8: track 0.00 -> 79.6 mm, vias 0 -> 5
- net /Right/COL_6: track 0.00 -> 32.0 mm, vias 0 -> 2
- net Net-(C303-Pad1): track 0.00 -> 1.85 mm

Commit message: just added a ground
Routing:
- net GND: track 116.7 -> 118.7 mm, vias 7 -> 8
Changed lines of the file:
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@@
   (via (at 307.987701 79.987701) (size 0.8) (drill 0.4) (layers "F.Cu" "B.Cu") (net 2))
   (via (at 54 83.5) (size 0.8) (drill 0.4) (layers "F.Cu" "B.Cu") (net 2))
+  (via (at 315.2 91.8) (size 0.8) (drill 0.4) (layers "F.Cu" "B.Cu") (net 2))
   (via (at 360 83.5) (size 0.8) (drill 0.4) (layers "F.Cu" "B.Cu") (net 2))
   (via (at 351 83.5) (size 0.8) (drill 0.4) (layers "F.Cu" "B.Cu") (net 2))
@@
   (segment (start 88.15 82.35) (end 87.9 82.35) (width 0.381) (layer "B.Cu") (net 2))
   (segment (start 64.973951 85.25) (end 70 85.25) (width 0.381) (layer "B.Cu") (net 2))
+  (segment (start 315.910589 91.089411) (end 315.2 91.8) (width 0.381) (layer "B.Cu") (net 2))
   (segment (start 63.6779 86.546051) (end 64.973951 85.25) (width 0.381) (layer "B.Cu") (net 2))
   (segment (start 325.639411 92.560589) (end 325.53454 92.560589) (width 0.381) (layer "B.Cu") (net 2))
@@
   (segment (start 307.575402 80.4) (end 306.1 80.4) (width 0.381) (layer "B.Cu") (net 2))
   (segment (start 325.52 77.25) (end 324.110399 77.25) (width 0.381) (layer "B.Cu") (net 2))
+  (segment (start 316.910589 91.089411) (end 315.910589 91.089411) (width 0.381) (layer "B.Cu") (net 2))
   (segment (start 325.53454 92.560589) (end 324.046051 91.0721) (width 0.381) (layer "B.Cu") (net 2))
   (segment (start 305.85 80.4) (end 306.1 80.4) (width 0.381) (layer "B.Cu") (net 2))
